Commit message: Adds namespacing

File: rover_demo_gz/urdf/drone.urdf.xacro (robot description, xacro)
@@ -4,9 +4,8 @@
   <xacro:property name="mass" value="1.0"/>
   <xacro:property name="arm_length" value="0.25"/>
-  <xacro:property name="link_prefix" value = "drone/" />
   <xacro:arg name="robot_ns" default=""/>
   <xacro:property name="robot_ns" value="$(arg robot_ns)"/>
   <!-- Base body -->
-  <link name="${link_prefix}base_link">
+  <link name="base_link">
     <inertial>
       <mass value="${mass}"/>
@@ -51,5 +50,5 @@
     </link>
     <joint name="${name}_joint" type="continuous">
-      <parent link="${link_prefix}base_link"/>
+      <parent link="base_link"/>
       <child link="${name}"/>
       <origin xyz="${x} ${y} 0" rpy="0 0 0"/>
@@ -59,10 +58,10 @@
   </xacro:macro>
   <!-- 4 rotors (alternating spin direction) -->
-  <xacro:rotor name="${link_prefix}rotor_fl" x="${arm_length}"  y="${arm_length}" />
-  <xacro:rotor name="${link_prefix}rotor_fr" x="${arm_length}"  y="-${arm_length}"/>
-  <xacro:rotor name="${link_prefix}rotor_rl" x="-${arm_length}" y="${arm_length}" />
-  <xacro:rotor name="${link_prefix}rotor_rr" x="-${arm_length}" y="-${arm_length}"/>
+  <xacro:rotor name="rotor_fl" x="${arm_length}"  y="${arm_length}" />
+  <xacro:rotor name="rotor_fr" x="${arm_length}"  y="-${arm_length}"/>
+  <xacro:rotor name="rotor_rl" x="-${arm_length}" y="${arm_length}" />
+  <xacro:rotor name="rotor_rr" x="-${arm_length}" y="-${arm_length}"/>
   <!-- IMU -->
-  <gazebo reference="${link_prefix}base_link">
+  <gazebo reference="base_link">
     <sensor type="imu" name="imu_sensor">
       <update_rate>100</update_rate>
@@ -76,6 +75,6 @@
     <plugin filename="gz-sim-multicopter-motor-model-system" name="gz::sim::systems::MulticopterMotorModel">
       <robotNamespace>${robot_ns}</robotNamespace>
-      <jointName>${link_prefix}rotor_fl_joint</jointName>
-      <linkName>${link_prefix}rotor_fl</linkName>
+      <jointName>rotor_fl_joint</jointName>
+      <linkName>rotor_fl</linkName>
       <turningDirection>ccw</turningDirection>
       <timeConstantUp>0.0125</timeConstantUp>
@@ -93,6 +92,6 @@
     <plugin filename="gz-sim-multicopter-motor-model-system" name="gz::sim::systems::MulticopterMotorModel">
       <robotNamespace>${robot_ns}</robotNamespace>
-      <jointName>${link_prefix}rotor_fr_joint</jointName>
-      <linkName>${link_prefix}rotor_fr</linkName>
+      <jointName>rotor_fr_joint</jointName>
+      <linkName>rotor_fr</linkName>
       <turningDirection>cw</turningDirection>
       <timeConstantUp>0.0125</timeConstantUp>
@@ -110,6 +109,6 @@
     <plugin filename="gz-sim-multicopter-motor-model-system" name="gz::sim::systems::MulticopterMotorModel">
       <robotNamespace>${robot_ns}</robotNamespace>
-      <jointName>${link_prefix}rotor_rl_joint</jointName>
-      <linkName>${link_prefix}rotor_rl</linkName>
+      <jointName>rotor_rl_joint</jointName>
+      <linkName>rotor_rl</linkName>
       <turningDirection>cw</turningDirection>
       <timeConstantUp>0.0125</timeConstantUp>
@@ -127,6 +126,6 @@
     <plugin filename="gz-sim-multicopter-motor-model-system" name="gz::sim::systems::MulticopterMotorModel">
       <robotNamespace>${robot_ns}</robotNamespace>
-      <jointName>${link_prefix}rotor_rr_joint</jointName>
-      <linkName>${link_prefix}rotor_rr</linkName>
+      <jointName>rotor_rr_joint</jointName>
+      <linkName>rotor_rr</linkName>
       <turningDirection>ccw</turningDirection>
       <timeConstantUp>0.0125</timeConstantUp>
@@ -147,5 +146,5 @@
         <commandSubTopic>cmd_vel</commandSubTopic>
         <enableSubTopic>velocity_controller/enable</enableSubTopic>
-        <comLinkName>${link_prefix}base_link</comLinkName>
+        <comLinkName>base_link</comLinkName>
         <velocityGain>3.3 3.3 3.5</velocityGain>
         <attitudeGain>5.0 5.0 0.9</attitudeGain>
@@ -160,5 +159,5 @@
         <rotorConfiguration>
           <rotor>
-            <jointName>${link_prefix}rotor_fl_joint</jointName>
+            <jointName>rotor_fl_joint</jointName>
             <forceConstant>8.54858e-06</forceConstant>
             <momentConstant>0.016</momentConstant>
@@ -166,5 +165,5 @@
           </rotor>
           <rotor>
-            <jointName>${link_prefix}rotor_fr_joint</jointName>
+            <jointName>rotor_fr_joint</jointName>
             <forceConstant>8.54858e-06</forceConstant>
             <momentConstant>0.016</momentConstant>
@@ -172,5 +171,5 @@
           </rotor>
           <rotor>
-            <jointName>${link_prefix}rotor_rl_joint</jointName>
+            <jointName>rotor_rl_joint</jointName>
             <forceConstant>8.54858e-06</forceConstant>
             <momentConstant>0.016</momentConstant>
@@ -178,5 +177,5 @@
           </rotor>
           <rotor>
-            <jointName>${link_prefix}rotor_rr_joint</jointName>
+            <jointName>rotor_rr_joint</jointName>
             <forceConstant>8.54858e-06</forceConstant>
             <momentConstant>0.016</momentConstant>
@@ -189,6 +188,7 @@
         <odom_topic>${robot_ns}/true_pose</odom_topic>
         <odom_frame>odom</odom_frame>
-        <robot_base_frame>${link_prefix}base_link</robot_base_frame>
-        <tf_topic>tf</tf_topic>
+        <dimensions>3</dimensions>
+        <robot_base_frame>base_link</robot_base_frame>
+        <tf_topic>${robot_ns}/tf</tf_topic>
     </plugin>
   </gazebo>

File: rover_demo_gz/urdf/macros.xacro (robot description, xacro)
@@ -5,10 +5,8 @@
                        rockers_fixed:=true
                        footprint_link:=true
-                       link_prefix:=''
-                       joint_prefix:=''
                        imu_translation:='0.0628 -0.0314 -0.0393'
                        mecanum_wheels:=false">
     <xacro:macro name="rocker_link" params="name">
-      <link name="${link_prefix}rocker_${name}_link">
+      <link name="rocker_${name}_link">
         <inertial>
           <mass value="1.387336"/>
@@ -32,5 +30,5 @@
     </xacro:macro>
     <xacro:macro name="wheel_link" params="name model">
-      <link name="${link_prefix}wheel_${name}_link">
+      <link name="wheel_${name}_link">
         <inertial>
           <mass value="0.283642"/>
@@ -66,5 +64,5 @@
     </xacro:macro>
     <xacro:macro name="mecanum_wheel_link" params="name model">
-      <link name="${link_prefix}wheel_${name}_link">
+      <link name="wheel_${name}_link">
         <inertial>
           <mass value="0.672214"/>
@@ -95,7 +93,7 @@
     <!-- LINKS -->
     <xacro:if value="${footprint_link}">
-      <link name="${link_prefix}base_footprint"/>
-    </xacro:if>
-    <link name="${link_prefix}base_link">
+      <link name="base_footprint"/>
+    </xacro:if>
+    <link name="base_link">
       <pose>0 0 0.19783 0 0 0</pose>
       <inertial>
@@ -133,5 +131,5 @@
     </xacro:unless>
     <xacro:if value="${default_antenna}">
-      <link name="${link_prefix}antenna_link">
+      <link name="antenna_link">
         <inertial>
           <mass value="0.001237"/>
@@ -155,54 +153,14 @@
       </link>
     </xacro:if>
-    <link name="${link_prefix}camera_frame"/>
-    <link name="${link_prefix}lidar_frame"/>
-    <link name="${link_prefix}camera_optical_frame"/>
-    <link name="${link_prefix}imu_frame"/>
-    <link name="${joint_prefix}rotor_FL_link">
-      <inertial>
-        <mass value="0.1"/>
-        <origin xyz="0 0 0"/>
-        <inertia
-          ixx="0.0001" ixy="0" ixz="0"
-          iyy="0.0001" iyz="0"
-          izz="0.0001"/>
-      </inertial>
-    </link>
-    <link name="${joint_prefix}rotor_FR_link">
-      <inertial>
-        <mass value="0.1"/>
-        <origin xyz="0 0 0"/>
-        <inertia
-          ixx="0.0001" ixy="0" ixz="0"
-          iyy="0.0001" iyz="0"
-          izz="0.0001"/>
-      </inertial>
-    </link>
-    <link name="${joint_prefix}rotor_RL_link">
-      <inertial>
-        <mass value="0.1"/>
-        <origin xyz="0 0 0"/>
-        <inertia
-          ixx="0.0001" ixy="0" ixz="0"
-          iyy="0.0001" iyz="0"
-          izz="0.0001"/>
-      </inertial>
-    </link>
-    <link name="${joint_prefix}rotor_RR_link">
-      <inertial>
-        <mass value="0.1"/>
-        <origin xyz="0 0 0"/>
-        <inertia
-          ixx="0.0001" ixy="0" ixz="0"
-          iyy="0.0001" iyz="0"
-          izz="0.0001"/>
-      </inertial>
-    </link>
+    <link name="camera_frame"/>
+    <link name="lidar_frame"/>
+    <link name="camera_optical_frame"/>
+    <link name="imu_frame"/>
     <!-- JOINTS -->
     <xacro:if value="${footprint_link}">
-      <joint name="${joint_prefix}base_joint" type="fixed">
+      <joint name="base_joint" type="fixed">
         <origin xyz="0 0 0.19783" rpy="0 0 0"/>
-        <parent link="${link_prefix}base_footprint"/>
-        <child link="${link_prefix}base_link"/>
+        <parent link="base_footprint"/>
+        <child link="base_link"/>
       </joint>
     </xacro:if>
@@ -213,22 +171,22 @@
       <xacro:property name="rockers_joint_type" value="revolute"/>
     </xacro:unless>
-    <joint name="${joint_prefix}rocker_L_joint" type="${rockers_joint_type}">
+    <joint name="rocker_L_joint" type="${rockers_joint_type}">
       <origin xyz="0.00263 0.14167 -0.04731" rpy="0 0 ${pi}"/>
-      <parent link="${link_prefix}base_link"/>
-      <child link="${link_prefix}rocker_L_link"/>
+      <parent link="base_link"/>
+      <child link="rocker_L_link"/>
       <axis xyz="0 1 0"/>
       <limit effort="100.0" lower="-0.24" upper="0.24" velocity="100.0"/>
       <dynamics friction="1.0" damping="0.1"/>
     </joint>
-    <joint name="${joint_prefix}rocker_R_joint" type="${rockers_joint_type}">
+    <joint name="rocker_R_joint" type="${rockers_joint_type}">
       <origin xyz="0.00263 -0.14167 -0.04731" rpy="0 0 0"/>
-      <parent link="${link_prefix}base_link"/>
-      <child link="${link_prefix}rocker_R_link"/>
+      <parent link="base_link"/>
+      <child link="rocker_R_link"/>
       <axis xyz="0 1 0"/>
       <limit effort="100.0" lower="-0.24" upper="0.24" velocity="100.0"/>
       <dynamics friction="1.0" damping="0.1"/>
-      <mimic joint="${joint_prefix}rocker_L_joint"/>
-    </joint>
-    <joint name="${joint_prefix}wheel_FL_joint" type="continuous">
+      <mimic joint="rocker_L_joint"/>
+    </joint>
+    <joint name="wheel_FL_joint" type="continuous">
       <xacro:if value="${mecanum_wheels}">
         <origin xyz="-0.15256 -0.00884 -0.08802" rpy="0 0 0"/>
@@ -237,11 +195,11 @@
         <origin xyz="-0.15256 -0.08214 -0.08802" rpy="0 0 0"/>
       </xacro:unless>
-      <parent link="${link_prefix}rocker_L_link"/>
-      <child link="${link_prefix}wheel_FL_link"/>
+      <parent link="rocker_L_link"/>
+      <child link="wheel_FL_link"/>
       <axis xyz="0 -1 0"/>
       <limit effort="2.0" velocity="6.0"/>
       <dynamics friction="0.3125" damping="0.1"/>
     </joint>
-    <joint name="${joint_prefix}wheel_RL_joint" type="continuous">
+    <joint name="wheel_RL_joint" type="continuous">
       <xacro:if value="${mecanum_wheels}">
         <origin xyz="0.15256 -0.00884 -0.08802" rpy="0 0 0"/>
@@ -250,11 +208,11 @@
         <origin xyz="0.15256 -0.08214 -0.08802" rpy="0 0 0"/>
       </xacro:unless>
-      <parent link="${link_prefix}rocker_L_link"/>
-      <child link="${link_prefix}wheel_RL_link"/>
+      <parent link="rocker_L_link"/>
+      <child link="wheel_RL_link"/>
       <axis xyz="0 -1 0"/>
       <limit effort="2.0" velocity="6.0"/>
       <dynamics friction="0.3125" damping="0.1"/>
     </joint>
-    <joint name="${joint_prefix}wheel_FR_joint" type="continuous">
+    <joint name="wheel_FR_joint" type="continuous">
       <xacro:if value="${mecanum_wheels}">
         <origin xyz="0.15256 -0.00884 -0.08802" rpy="0 0 0"/>
@@ -263,11 +221,11 @@
         <origin xyz="0.15256 -0.08214 -0.08802" rpy="0 0 0"/>
       </xacro:unless>
-      <parent link="${link_prefix}rocker_R_link"/>
-      <child link="${link_prefix}wheel_FR_link"/>
+      <parent link="rocker_R_link"/>
+      <child link="wheel_FR_link"/>
       <axis xyz="0 1 0"/>
       <limit effort="2.0" velocity="6.0"/>
       <dynamics friction="0.3125" damping="0.1"/>
     </joint>
-    <joint name="${joint_prefix}wheel_RR_joint" type="continuous">
+    <joint name="wheel_RR_joint" type="continuous">
       <xacro:if value="${mecanum_wheels}">
         <origin xyz="-0.15256 -0.00884 -0.08802" rpy="0 0 0"/>
@@ -276,6 +234,6 @@
         <origin xyz="-0.15256 -0.08214 -0.08802" rpy="0 0 0"/>
       </xacro:unless>
-      <parent link="${link_prefix}rocker_R_link"/>
-      <child link="${link_prefix}wheel_RR_link"/>
+      <parent link="rocker_R_link"/>
+      <child link="wheel_RR_link"/>
       <axis xyz="0 1 0"/>
       <limit effort="2.0" velocity="6.0"/>
@@ -283,62 +241,36 @@
     </joint>
     <xacro:if value="${default_antenna}">
-      <joint name="${joint_prefix}antenna_joint" type="fixed">
+      <joint name="antenna_joint" type="fixed">
         <origin xyz="-0.0052 0.056 -0.0065" rpy="0 0 0"/>
-        <parent link="${link_prefix}base_link"/>
-        <child link="${link_prefix}antenna_link"/>
+        <parent link="base_link"/>
+        <child link="antenna_link"/>
       </joint>
     </xacro:if>
-    <joint name="${joint_prefix}lidar_joint" type="fixed">
+    <joint name="lidar_joint" type="fixed">
       <origin xyz="0.0971 0 -0.0427" rpy="0 0.2094 0"/>
-      <parent link="${link_prefix}base_link"/>
-      <child link="${link_prefix}lidar_frame"/>
-    </joint>
-    <joint name="${joint_prefix}camera_joint" type="fixed">
+      <parent link="base_link"/>
+      <child link="lidar_frame"/>
+    </joint>
+    <joint name="camera_joint" type="fixed">
       <origin xyz="0.0971 0 -0.0427" rpy="0 0.2094 0"/>
-      <parent link="${link_prefix}base_link"/>
-      <child link="${link_prefix}camera_frame"/>
-    </joint>
-    <joint name="${joint_prefix}camera_optical_joint" type="fixed">
+      <parent link="base_link"/>
+      <child link="camera_frame"/>
+    </joint>
+    <joint name="camera_optical_joint" type="fixed">
       <origin xyz="0 0 0" rpy="-${pi/2} 0.0 -${pi/2}"/>
-      <parent link="${link_prefix}camera_frame"/>
-      <child link="${link_prefix}camera_optical_frame"/>
-    </joint>
-    <joint name="${joint_prefix}imu_joint" type="fixed">
+      <parent link="camera_frame"/>
+      <child link="camera_optical_frame"/>
+    </joint>
+    <joint name="imu_joint" type="fixed">
       <origin xyz="${imu_translation}" rpy="0 0 0"/>
-      <parent link="${link_prefix}base_footprint"/>
-      <child link="${link_prefix}imu_frame"/>
-    </joint>
-    <joint name="${joint_prefix}rotor_FL_joint" type="continuous">
-      <parent link="${link_prefix}base_link"/>
-      <child link="${link_prefix}rotor_FL_link"/>
-      <origin xyz="0.2 0.2 0.1" rpy="0 0 0"/>
-      <axis xyz="0 0 1"/>
-    </joint>
-    <joint name="${joint_prefix}rotor_FR_joint" type="continuous">
-      <parent link="${link_prefix}base_link"/>
-      <child link="${link_prefix}rotor_FR_link"/>
-      <origin xyz="0.2 -0.2 0.1" rpy="0 0 0"/>
-      <axis xyz="0 0 1"/>
-    </joint>
-    <joint name="${joint_prefix}rotor_RL_joint" type="continuous">
-      <parent link="${link_prefix}base_link"/>
-      <child link="${link_prefix}rotor_RL_link"/>
-      <origin xyz="-0.2 0.2 0.1" rpy="0 0 0"/>
-      <axis xyz="0 0 1"/>
-    </joint>
-    <joint name="${joint_prefix}rotor_RR_joint" type="continuous">
-      <parent link="${link_prefix}base_link"/>
-      <child link="${link_prefix}rotor_RR_link"/>
-      <origin xyz="-0.2 -0.2 0.1" rpy="0 0 0"/>
-      <axis xyz="0 0 1"/>
+      <parent link="base_footprint"/>
+      <child link="imu_frame"/>
     </joint>
   </xacro:macro>
   <!-- LEO GAZEBO -->
   <xacro:macro name="leo_gazebo"
-               params="robot_ns:=''
-               link_prefix:=''
-               joint_prefix:=''">
+               params="robot_ns:=''">
     <!-- base ODE properties -->
-    <gazebo reference="${link_prefix}base_footprint">
+    <gazebo reference="base_footprint">
       <collision>
         <surface>
@@ -357,5 +289,5 @@
       </collision>
     </gazebo>
-    <gazebo reference="${link_prefix}base_link">
+    <gazebo reference="base_link">
       <collision>
         <surface>
@@ -375,5 +307,5 @@
     </gazebo>
     <!-- rocker ODE properties -->
-    <gazebo reference="${link_prefix}rocker_L_link">
+    <gazebo reference="rocker_L_link">
       <collision>
         <surface>
@@ -392,5 +324,5 @@
       </collision>
     </gazebo>
-    <gazebo reference="${link_prefix}rocker_R_link">
+    <gazebo reference="rocker_R_link">
       <collision>
         <surface>
@@ -410,5 +342,5 @@
     </gazebo>
     <!-- wheel ODE properties -->
-    <gazebo reference="${link_prefix}wheel_FL_link">
+    <gazebo reference="wheel_FL_link">
       <collision>
         <surface>
@@ -429,5 +361,5 @@
       </collision>
     </gazebo>
-    <gazebo reference="${link_prefix}wheel_FR_link">
+    <gazebo reference="wheel_FR_link">
       <collision>
         <surface>
@@ -448,5 +380,5 @@
       </collision>
     </gazebo>
-    <gazebo reference="${link_prefix}wheel_RL_link">
+    <gazebo reference="wheel_RL_link">
       <collision>
         <surface>
@@ -467,5 +399,5 @@
       </collision>
     </gazebo>
-    <gazebo reference="${link_prefix}wheel_RR_link">
+    <gazebo reference="wheel_RR_link">
       <collision>
         <surface>
@@ -487,5 +419,5 @@
     </gazebo>
     <!-- camera -->
-    <gazebo reference="${link_prefix}camera_frame">
+    <gazebo reference="camera_frame">
       <sensor name="camera" type="camera">
           <camera name="leo_camera">
@@ -517,13 +449,13 @@
           <update_rate>30</update_rate>
           <visualize>true</visualize>
-          <topic>${link_prefix}camera/image_raw</topic>
-          <gz_frame_id>${link_prefix}camera_frame</gz_frame_id>
+          <topic>${robot_ns}/camera/image_raw</topic>
+          <gz_frame_id>camera_frame</gz_frame_id>
       </sensor>
     </gazebo>
     <!-- fake lidar for sim-->
-    <gazebo reference="${link_prefix}lidar_frame">
+    <gazebo reference="lidar_frame">
       <sensor name='lidar_frame' type='gpu_lidar'>
         <pose relative_to='lidar_frame'>0 0 0 0 0 0</pose>
-        <topic>${link_prefix}pointcloud</topic>
+        <topic>${robot_ns}/pointcloud</topic>
         <update_rate>10</update_rate>
         <ray>
@@ -550,5 +482,5 @@
         <always_on>true</always_on>
         <visualize>true</visualize>
-        <gz_frame_id>${link_prefix}lidar_frame</gz_frame_id>
+        <gz_frame_id>lidar_frame</gz_frame_id>
       </sensor>
     </gazebo>
@@ -556,6 +488,6 @@
     <gazebo>
       <plugin name="leo_gz::DifferentialSystem" filename="libleo_gz_differential_plugin.so">
-        <jointA>${joint_prefix}rocker_L_joint</jointA>
-        <jointB>${joint_prefix}rocker_R_joint</jointB>
+        <jointA>rocker_L_joint</jointA>
+        <jointB>rocker_R_joint</jointB>
         <forceConstant>100.0</forceConstant>
       </plugin>
@@ -565,14 +497,14 @@
         filename="ignition-gazebo-joint-state-publisher-system"
         name="ignition::gazebo::systems::JointStatePublisher">
-        <topic>${link_prefix}joint_states</topic>
+        <topic>${robot_ns}/joint_states</topic>
       </plugin>
     </gazebo>
-    <gazebo reference="${link_prefix}imu_frame">
+    <gazebo reference="imu_frame">
       <sensor type="imu" name="leo_imu_sensor">
         <update_rate>100</update_rate>
         <visualize>true</visualize>
-        <topic>${link_prefix}imu/data_raw</topic>
+        <topic>${robot_ns}/imu/data_raw</topic>
         <always_on>1</always_on>
-        <gz_frame_id>${link_prefix}imu_frame</gz_frame_id>
+        <gz_frame_id>imu_frame</gz_frame_id>
       </sensor>
     </gazebo>
@@ -581,12 +513,12 @@
         filename="libignition-gazebo-diff-drive-system.so"
         name="ignition::gazebo::systems::DiffDrive">
-        <left_joint>${joint_prefix}wheel_FL_joint</left_joint>
-        <right_joint>${joint_prefix}wheel_FR_joint</right_joint>
-        <left_joint>${joint_prefix}wheel_RL_joint</left_joint>
-        <right_joint>${joint_prefix}wheel_RR_joint</right_joint>
+        <left_joint>wheel_FL_joint</left_joint>
+        <right_joint>wheel_FR_joint</right_joint>
+        <left_joint>wheel_RL_joint</left_joint>
+        <right_joint>wheel_RR_joint</right_joint>
         <wheel_separation>0.358</wheel_separation>
         <wheel_radius>0.0625</wheel_radius>
         <frame_id>odom</frame_id>
-        <child_frame_id>${link_prefix}base_footprint</child_frame_id>
+        <child_frame_id>base_footprint</child_frame_id>
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