Commit message: Update namespacing

File: rover_demo_gz/urdf/drone.urdf.xacro (robot description, xacro)
@@ -188,5 +188,5 @@
         <odom_topic>${robot_ns}/true_pose</odom_topic>
         <odom_frame>odom</odom_frame>
-        <dimensions>3</dimensions>
+        <dimensions>2</dimensions>
         <robot_base_frame>base_link</robot_base_frame>
         <tf_topic>${robot_ns}/tf</tf_topic>

File: rover_demo_gz/urdf/macros.xacro (robot description, xacro)
@@ -4,5 +4,4 @@
                params="default_antenna:=true
                        rockers_fixed:=true
-                       footprint_link:=true
                        imu_translation:='0.0628 -0.0314 -0.0393'
                        mecanum_wheels:=false">
@@ -92,7 +91,4 @@
     </xacro:macro>
     <!-- LINKS -->
-    <xacro:if value="${footprint_link}">
-      <link name="base_footprint"/>
-    </xacro:if>
     <link name="base_link">
       <pose>0 0 0.19783 0 0 0</pose>
@@ -158,11 +154,4 @@
     <link name="imu_frame"/>
     <!-- JOINTS -->
-    <xacro:if value="${footprint_link}">
-      <joint name="base_joint" type="fixed">
-        <origin xyz="0 0 0.19783" rpy="0 0 0"/>
-        <parent link="base_footprint"/>
-        <child link="base_link"/>
-      </joint>
-    </xacro:if>
     <xacro:if value="${rockers_fixed}">
       <xacro:property name="rockers_joint_type" value="fixed"/>
@@ -264,5 +253,5 @@
     <joint name="imu_joint" type="fixed">
       <origin xyz="${imu_translation}" rpy="0 0 0"/>
-      <parent link="base_footprint"/>
+      <parent link="base_link"/>
       <child link="imu_frame"/>
     </joint>
@@ -272,5 +261,5 @@
                params="robot_ns:=''">
     <!-- base ODE properties -->
-    <gazebo reference="base_footprint">
+    <gazebo reference="base_link">
       <collision>
         <surface>
@@ -520,5 +509,5 @@
         <wheel_radius>0.0625</wheel_radius>
         <frame_id>odom</frame_id>
-        <child_frame_id>base_footprint</child_frame_id>
+        <child_frame_id>base_link</child_frame_id>
         <odom_publish_frequency>20</odom_publish_frequency>
         <topic>${robot_ns}/cmd_vel</topic>
@@ -532,6 +521,6 @@
         <odom_topic>${robot_ns}/true_pose</odom_topic>
         <odom_frame>odom</odom_frame>
-        <dimensions>3</dimensions>
-        <robot_base_frame>base_footprint</robot_base_frame>
+        <dimensions>2</dimensions>
+        <robot_base_frame>base_link</robot_base_frame>
         <tf_topic>${robot_ns}/tf</tf_topic>
       </plugin>
@@ -551,5 +540,5 @@
       <joint name="fixed" type="fixed">
         <parent link="odom"/>
-        <child link="base_footprint"/>
+        <child link="base_link"/>
         <origin xyz="0.0 0.0 1.0"/>
       </joint>
