Commit message: Adds setup for multimodal robot

File: rover_demo_gz/urdf/macros.xacro (robot description, xacro)
@@ -237,5 +237,5 @@
     </xacro:if>
     <joint name="lidar_joint" type="fixed">
-      <origin xyz="0.0971 0 -0.0427" rpy="0 0.2094 0"/>
+      <origin xyz="0.0971 0 -0.0427" rpy="0 0.7 0"/>
       <parent link="base_link"/>
       <child link="lidar_frame"/>
@@ -448,5 +448,5 @@
         <topic>${robot_ns}/pointcloud</topic>
         <update_rate>10</update_rate>
-        <ray>
+        <lidar>
           <scan>
             <horizontal>
@@ -464,22 +464,22 @@
           </scan>
           <range>
-            <min>1.0</min>
-            <max>10.0</max>
+            <min>0.5</min>
+            <max>2.0</max>
             <resolution>0.01</resolution>
           </range>
-        </ray>
+        </lidar>
         <always_on>true</always_on>
         <visualize>true</visualize>
         <gz_frame_id>lidar_frame</gz_frame_id>
       </sensor>
+      <plugin name="lidar_plugin" filename="libgazebo_ros_laser.so">
+        <ros>
+          <namespace>${robot_ns}</namespace>
+          <parameter name="frame_id" value="lidar_frame"/>
+          <topic>pointcloud</topic>
+        </ros>
+      </plugin>
     </gazebo>
     <!-- rocker differential -->
-    <gazebo>
-      <plugin name="leo_gz::DifferentialSystem" filename="libleo_gz_differential_plugin.so">
-        <jointA>rocker_L_joint</jointA>
-        <jointB>rocker_R_joint</jointB>
-        <forceConstant>100.0</forceConstant>
-      </plugin>
-    </gazebo>
     <gazebo>
       <plugin
@@ -521,5 +521,5 @@
         <odom_topic>${robot_ns}/true_pose</odom_topic>
         <odom_frame>odom</odom_frame>
-        <dimensions>2</dimensions>
+        <dimensions>3</dimensions>
         <robot_base_frame>base_link</robot_base_frame>
         <tf_topic>${robot_ns}/tf</tf_topic>

File: rover_demo_gz/urdf/multimodal.urdf.xacro (robot description, xacro)
@@ -1,37 +1,63 @@
 <?xml version="1.0"?>
-<robot xmlns:xacro="http://www.ros.org/wiki/xacro" name="drone">
-  <!-- Parameters -->
-  <xacro:property name="mass" value="1.0"/>
+<robot xmlns:xacro="http://www.ros.org/wiki/xacro" name="cube_bot">
+  <xacro:property name="cube_size" value="0.4"/>
+  <xacro:property name="wheel_radius" value="0.1"/>
+  <xacro:property name="wheel_width" value="0.05"/>
+  <xacro:property name="link_prefix" value="cube/"/>
+  <xacro:property name="mast_height" value="0.1"/>
   <xacro:property name="arm_length" value="0.25"/>
   <xacro:arg name="robot_ns" default=""/>
   <xacro:property name="robot_ns" value="$(arg robot_ns)"/>
-  <!-- Base body -->
   <link name="base_link">
-    <inertial>
-      <mass value="${mass}"/>
-      <origin xyz="0 0 0" rpy="0 0 0"/>
-      <inertia ixx="0.02" ixy="0" ixz="0"
-               iyy="0.02" iyz="0"
-               izz="0.04"/>
-    </inertial>
     <visual>
       <geometry>
-        <cylinder radius="0.12" length="0.05"/>
+        <box size="${cube_size} ${cube_size} ${cube_size/2}"/>
       </geometry>
-      <origin xyz="0 0 0" rpy="0 0 0"/>
+      <material name="cube_color">
+        <color rgba="0.2 0.2 0.2 1.0"/>
+      </material>
     </visual>
     <collision>
       <geometry>
-        <cylinder radius="0.12" length="0.05"/>
+        <box size="${cube_size} ${cube_size} ${cube_size/2}"/>
       </geometry>
-      <origin xyz="0 0 0" rpy="0 0 0"/>
     </collision>
+    <inertial>
+      <mass value="0.1"/>
+      <inertia ixx="0.2" ixy="0.0" ixz="0.0" iyy="0.2" iyz="0.0" izz="0.2"/>
+    </inertial>
   </link>
-  <link name="camera_frame"/>
-  <link name="lidar_frame"/>
-  <link name="camera_optical_frame"/>
-  <!-- Rotor macro -->
+  <xacro:macro name="wheel" params="name x y side">
+    <link name="${name}_link">
+      <visual>
+        <origin rpy="1.5708 0 0"/>
+        <geometry>
+          <cylinder radius="${wheel_radius}" length="${wheel_width}"/>
+        </geometry>
+        <material name="black">
+          <color rgba="0 0 0 1"/>
+        </material>
+      </visual>
+      <collision>
+        <origin rpy="1.5708 0 0"/>
+        <geometry>
+          <cylinder radius="${wheel_radius}" length="${wheel_width}"/>
+        </geometry>
+      </collision>
+      <inertial>
+        <mass value="0.1"/>
+        <inertia ixx="0.01" ixy="0.0" ixz="0.0" iyy="0.01" iyz="0.0" izz="0.01"/>
+      </inertial>
+    </link>
+    <joint name="${name}_joint" type="continuous">
+      <parent link="base_link"/>
+      <child link="${name}_link"/>
+      <origin
+        xyz="${x} ${y + side * (cube_size/2 + wheel_width/2)} ${-cube_size/4 + wheel_radius -0.1}"/>
+      <axis xyz="0 1 0"/>
+    </joint>
+  </xacro:macro>
   <xacro:macro name="rotor" params="name x y">
-    <link name="${name}">
+    <link name="${name}_link">
       <inertial>
         <mass value="0.05"/>
@@ -43,10 +69,10 @@
       <visual>
         <geometry>
-          <cylinder radius="0.05" length="0.01"/>
+          <cylinder radius="0.1" length="0.01"/>
         </geometry>
       </visual>
       <collision>
         <geometry>
-          <cylinder radius="0.05" length="0.01"/>
+          <cylinder radius="0.1" length="0.01"/>
         </geometry>
       </collision>
@@ -54,45 +80,124 @@
     <joint name="${name}_joint" type="continuous">
       <parent link="base_link"/>
-      <child link="${name}"/>
-      <origin xyz="${x} ${y} 0" rpy="0 0 0"/>
+      <child link="${name}_link"/>
+      <origin xyz="${x} ${y} ${cube_size / 4 + 0.05}" rpy="0 0 0"/>
       <axis xyz="0 0 1"/>
       <limit effort="10.0" velocity="500.0"/>
     </joint>
   </xacro:macro>
-  <joint name="lidar_joint" type="fixed">
-    <origin xyz="0.0 0.0 -0.1" rpy="0.0 1.57 0.0"/>
-    <parent link="base_link"/>
-    <child link="lidar_frame"/>
-  </joint>
-  <joint name="camera_joint" type="fixed">
-    <origin xyz="0.0 0.0 -0.1" rpy="0.0 1.57 0.0"/>
-    <parent link="base_link"/>
-    <child link="camera_frame"/>
-  </joint>
-  <joint name="camera_optical_joint" type="fixed">
-    <origin xyz="0 0 0" rpy="-${pi/2} 0.0 -${pi/2}"/>
-    <parent link="camera_frame"/>
-    <child link="camera_optical_frame"/>
-  </joint>
-  <!-- 4 rotors (alternating spin direction) -->
+  <xacro:wheel name="wheel_fl"
+               x="${ cube_size/2}"
+               y="${ 0}"
+               side="1"/>
+  <xacro:wheel name="wheel_rl"
+               x="${-cube_size/2}"
+               y="${ 0}"
+               side="1"/>
+  <xacro:wheel name="wheel_fr"
+               x="${ cube_size/2}"
+               y="${ 0}"
+               side="-1"/>
+  <xacro:wheel name="wheel_rr"
+               x="${-cube_size/2}"
+               y="${ 0}"
+               side="-1"/>
   <xacro:rotor name="rotor_fl" x="${arm_length}"  y="${arm_length}" />
   <xacro:rotor name="rotor_fr" x="${arm_length}"  y="-${arm_length}"/>
   <xacro:rotor name="rotor_rl" x="-${arm_length}" y="${arm_length}" />
   <xacro:rotor name="rotor_rr" x="-${arm_length}" y="-${arm_length}"/>
-  <!-- IMU -->
-  <gazebo reference="base_link">
-    <sensor type="imu" name="imu_sensor">
-      <update_rate>100</update_rate>
+  <link name="mast_link">
+    <visual>
+      <origin xyz="0 0 ${mast_height/2}"/>
+      <geometry>
+        <cylinder radius="0.03" length="${mast_height}"/>
+      </geometry>
+      <material name="black">
+        <color rgba="0 0 0 1"/>
+      </material>
+    </visual>
+    <collision>
+      <origin xyz="0 0 ${mast_height/2}"/>
+      <geometry>
+        <cylinder radius="0.03" length="${mast_height}"/>
+      </geometry>
+    </collision>
+    <inertial>
+      <mass value="0.1"/>
+      <inertia ixx="0.01" ixy="0.0" ixz="0.0" iyy="0.01" iyz="0.0" izz="0.01"/>
+    </inertial>
+  </link>
+  <joint name="mast_joint" type="fixed">
+    <parent link="base_link"/>
+    <child link="mast_link"/>
+    <origin xyz="0 0 ${cube_size/2}"/>
+  </joint>
+  <link name="camera_link"/>
+  <link name="lidar_link"/>
+<joint name="camera_joint" type="fixed">
+  <parent link="mast_link"/>
+  <child link="camera_link"/>
+  <origin xyz="0.02 0 ${mast_height}" rpy="0 0 1.5708"/>
+</joint>
+<joint name="lidar_joint" type="fixed">
+  <parent link="mast_link"/>
+  <child link="lidar_link"/>
+  <origin xyz="0.02 0 ${mast_height}" rpy="0 0 1.5708"/>
+</joint>
+<!-- Sensors -->
+  <gazebo reference="camera_link">
+    <sensor name="camera" type="camera">
+      <camera name="cube_camera">
+        <horizontal_fov>1.9</horizontal_fov>
+        <image>
+          <width>640</width>
+          <height>480</height>
+          <format>R8G8B8</format>
+        </image>
+        <clip>
+          <near>0.2</near>
+          <far>300</far>
+        </clip>
+      </camera>
       <always_on>1</always_on>
+      <update_rate>30</update_rate>
       <visualize>true</visualize>
-      <topic>${robot_ns}/imu/data_raw</topic>
+      <topic>camera/image_raw</topic>
+      <gz_frame_id>camera_link</gz_frame_id>
     </sensor>
   </gazebo>
-  <!-- Plugins -->
+  <gazebo reference="lidar_link">
+    <sensor name="lidar_link" type="gpu_lidar">
+    <pose>0 0 0 0 0 0</pose>
+      <topic>pointcloud</topic>
+      <update_rate>10</update_rate>
+      <ray>
+        <scan>
+          <horizontal>
+            <samples>640</samples>
+            <min_angle>-1.396263</min_angle>
+            <max_angle>1.396263</max_angle>
+          </horizontal>
+          <vertical>
+            <samples>32</samples>
+            <min_angle>-1.39</min_angle>
+            <max_angle>1.39</max_angle>
+          </vertical>
+        </scan>
+        <range>
+          <min>1.0</min>
+          <max>10.0</max>
+        </range>
+      </ray>
+      <always_on>true</always_on>
+      <visualize>true</visualize>
+      <gz_frame_id>lidar_link</gz_frame_id>
+    </sensor>
+  </gazebo>
+  <!-- Motion plugins -->
   <gazebo>
     <plugin filename="gz-sim-multicopter-motor-model-system" name="gz::sim::systems::MulticopterMotorModel">
       <robotNamespace>${robot_ns}</robotNamespace>
       <jointName>rotor_fl_joint</jointName>
-      <linkName>rotor_fl</linkName>
+      <linkName>rotor_fl_link</linkName>
       <turningDirection>ccw</turningDirection>
       <timeConstantUp>0.0125</timeConstantUp>
@@ -111,5 +216,5 @@
       <robotNamespace>${robot_ns}</robotNamespace>
       <jointName>rotor_fr_joint</jointName>
-      <linkName>rotor_fr</linkName>
+      <linkName>rotor_fr_link</linkName>
       <turningDirection>cw</turningDirection>
       <timeConstantUp>0.0125</timeConstantUp>
@@ -128,5 +233,5 @@
       <robotNamespace>${robot_ns}</robotNamespace>
       <jointName>rotor_rl_joint</jointName>
-      <linkName>rotor_rl</linkName>
+      <linkName>rotor_rl_link</linkName>
       <turningDirection>cw</turningDirection>
       <timeConstantUp>0.0125</timeConstantUp>
@@ -145,5 +250,5 @@
       <robotNamespace>${robot_ns}</robotNamespace>
       <jointName>rotor_rr_joint</jointName>
-      <linkName>rotor_rr</linkName>
+      <linkName>rotor_rr_link</linkName>
       <turningDirection>ccw</turningDirection>
       <timeConstantUp>0.0125</timeConstantUp>
@@ -162,5 +267,5 @@
         name="gz::sim::systems::MulticopterVelocityControl">
         <robotNamespace>${robot_ns}</robotNamespace>
-        <commandSubTopic>cmd_vel</commandSubTopic>
+        <commandSubTopic>cmd_vel_air</commandSubTopic>
         <enableSubTopic>velocity_controller/enable</enableSubTopic>
         <comLinkName>base_link</comLinkName>
@@ -202,4 +307,22 @@
         </rotorConfiguration>
     </plugin>
+    <plugin
+      filename="libignition-gazebo-diff-drive-system.so"
+      name="ignition::gazebo::systems::DiffDrive">
+      <left_joint>wheel_fl_joint</left_joint>
+      <right_joint>wheel_fr_joint</right_joint>
+      <left_joint>wheel_rl_joint</left_joint>
+      <right_joint>wheel_rr_joint</right_joint>
+      <wheel_separation>${cube_size}</wheel_separation>
+      <wheel_radius>${wheel_radius}</wheel_radius>
+      <frame_id>odom</frame_id>
+      <child_frame_id>base_link</child_frame_id>
+      <odom_publish_frequency>20</odom_publish_frequency>
+      <topic>${robot_ns}/cmd_vel_ground</topic>
+      <max_linear_acceleration>2.5</max_linear_acceleration>
+      <max_angular_acceleration>3</max_angular_acceleration>
+      <min_linear_acceleration>-2.5</min_linear_acceleration>
+      <min_angular_acceleration>-3</min_angular_acceleration>
+    </plugin>
     <plugin filename="libignition-gazebo-odometry-publisher-system.so" name="ignition::gazebo::systems::OdometryPublisher">
         <update_frequency>10</update_frequency>
@@ -211,69 +334,3 @@
     </plugin>
   </gazebo>
-     <gazebo reference="camera_frame">
-      <sensor name="camera" type="camera">
-          <camera name="drone_camera">
-              <horizontal_fov>1.9</horizontal_fov>
-              <image>
-                  <width>640</width>
-                  <height>480</height>
-                  <format>R8G8B8</format>
-              </image>
-              <clip>
-                  <near>0.2</near>
-                  <far>300</far>
-              </clip>
-              <noise>
-                <type>gaussian</type>
-                <mean>0.0</mean>
-                <stddev>0.007</stddev>
-              </noise>
-              <distortion>
-                <k1>-0.279817</k1>
-                <k2>0.060321</k2>
-                <k3>0.000487</k3>
-                <p1>0.000310</p1>
-                <p2>0.000000</p2>
-                <center>0.5 0.5</center>
-              </distortion>
-          </camera>
-          <always_on>1</always_on>
-          <update_rate>30</update_rate>
-          <visualize>true</visualize>
-          <topic>${robot_ns}/camera/image_raw</topic>
-          <gz_frame_id>camera_frame</gz_frame_id>
-      </sensor>
-    </gazebo>
-    <!-- fake lidar for sim-->
-    <gazebo reference="lidar_frame">
-      <sensor name='lidar_frame' type='gpu_lidar'>
-        <pose relative_to='lidar_frame'>0 0 0 0 0 0</pose>
-        <topic>${robot_ns}/pointcloud</topic>
-        <update_rate>10</update_rate>
-        <ray>
-          <scan>
-            <horizontal>
-              <samples>640</samples>
-              <resolution>1</resolution>
-              <min_angle>-1.396263</min_angle>
-              <max_angle>1.396263</max_angle>
-            </horizontal>
-            <vertical>
-              <samples>32</samples>
-              <resolution>0.01</resolution>
-              <min_angle>-1.39</min_angle>
-              <max_angle>1.39</max_angle>
-            </vertical>
-          </scan>
-          <range>
-            <min>1.0</min>
-            <max>10.0</max>
-            <resolution>0.01</resolution>
-          </range>
-        </ray>
-        <always_on>true</always_on>
-        <visualize>true</visualize>
-        <gz_frame_id>lidar_frame</gz_frame_id>
-      </sensor>
-    </gazebo>
 </robot>
