Commit message: Move robots into dedicated description packages

File: leo_description/urdf/leo.urdf.xacro (robot description, xacro)
@@ -3,5 +3,5 @@
        name="leo">
   <xacro:arg name="mecanum_wheels" default="false"/>
-  <xacro:include filename="$(find rover_demo_gz)/urdf/macros.xacro"/>
+  <xacro:include filename="$(find leo_description)/urdf/macros.xacro"/>
   <xacro:leo mecanum_wheels="$(arg mecanum_wheels)"/>
 </robot>

File: leo_description/urdf/leo_sim.urdf (robot description, URDF)
Before this commit: robot leo_sim, 17 links, 16 joints
Links:
- link antenna_link: geometry collision cylinder length=0.056 radius=0.0055; visual mesh filename=package://leo_description/models/Antenna.dae
- link base_link: geometry collision mesh filename=package://leo_description/models/Chassis_outline.stl; visual mesh filename=package://leo_description/models/Chassis.dae
- link rocker_L_link: geometry collision mesh filename=package://leo_description/models/Rocker_outline.stl; visual mesh filename=package://leo_description/models/Rocker.dae
- link rocker_R_link: geometry collision mesh filename=package://leo_description/models/Rocker_outline.stl; visual mesh filename=package://leo_description/models/Rocker.dae
- link wheel_FL_link: geometry collision cylinder length=0.04 radius=0.0625; collision cylinder length=0.07 radius=0.057
- link wheel_FR_link: geometry collision cylinder length=0.04 radius=0.0625; collision cylinder length=0.07 radius=0.057
- link wheel_RL_link: geometry collision cylinder length=0.04 radius=0.0625; collision cylinder length=0.07 radius=0.057
- link wheel_RR_link: geometry collision cylinder length=0.04 radius=0.0625; collision cylinder length=0.07 radius=0.057

File: leo_description/urdf/leo_sim.urdf.xacro (robot description, xacro)
@@ -5,5 +5,5 @@
   <xacro:arg name="robot_ns" default=""/>
   <xacro:arg name="mecanum_wheels" default="false"/>
-  <xacro:include filename="$(find rover_demo_gz)/urdf/macros.xacro"/>
+  <xacro:include filename="$(find leo_description)/urdf/macros.xacro"/>
   <xacro:leo_sim robot_ns="$(arg robot_ns)"
                  fixed="$(arg fixed)"

File: leo_description/urdf/macros.xacro (robot description, xacro)
@@ -18,10 +18,10 @@
         <visual>
           <geometry>
-            <mesh filename="package://leo/Rocker.dae"/>
+            <mesh filename="package://Rocker.dae"/>
           </geometry>
         </visual>
         <collision>
           <geometry>
-            <mesh filename="package://leo/Rocker_outline.stl"/>
+            <mesh filename="package://Rocker_outline.stl"/>
           </geometry>
         </collision>
@@ -40,5 +40,5 @@
         <visual>
           <geometry>
-            <mesh filename="package://leo/Wheel${model}.dae"/>
+            <mesh filename="package://Wheel${model}.dae"/>
           </geometry>
         </visual>
@@ -57,5 +57,5 @@
         <collision>
           <geometry>
-            <mesh filename="package://leo/Wheel_outline.stl"/>
+            <mesh filename="package://Wheel_outline.stl"/>
           </geometry>
         </collision>
@@ -74,5 +74,5 @@
         <visual>
           <geometry>
-            <mesh filename="package://leo/WheelMecanum${model}.dae"/>
+            <mesh filename="package://WheelMecanum${model}.dae"/>
           </geometry>
         </visual>
@@ -85,5 +85,5 @@
         <collision>
           <geometry>
-            <mesh filename="package://leo/Mecanum_wheel_outline.stl"/>
+            <mesh filename="package://Mecanum_wheel_outline.stl"/>
           </geometry>
         </collision>
@@ -103,10 +103,10 @@
       <visual>
         <geometry>
-          <mesh filename="package://leo/Chassis.dae"/>
+          <mesh filename="package://Chassis.dae"/>
         </geometry>
       </visual>
       <collision>
         <geometry>
-          <mesh filename="package://leo/Chassis_outline.stl"/>
+          <mesh filename="package://Chassis_outline.stl"/>
         </geometry>
       </collision>
@@ -138,5 +138,5 @@
         <visual>
           <geometry>
-            <mesh filename="package://leo/Antenna.dae"/>
+            <mesh filename="package://Antenna.dae"/>
           </geometry>
         </visual>
