Commit message: Go2 now spawns with ros control and champ

File: go2_description/urdf/const.xacro (robot description, xacro)
@@ -39,6 +39,6 @@
     <xacro:property name="calf_offset_z" value="-0.213"/>
     <!-- joint limits -->
-    <xacro:property name="damping" value="0.0"/>
-    <xacro:property name="friction" value="0.0"/>
+    <xacro:property name="damping" value="0.01"/>
+    <xacro:property name="friction" value="0.2"/>
     <xacro:property name="hip_position_max" value="1.0472"/>
     <xacro:property name="hip_position_min" value="-1.0472"/>

File: go2_description/urdf/leg.xacro (robot description, xacro)
@@ -1,5 +1,5 @@
 <?xml version="1.0"?>
 <robot xmlns:xacro="http://www.ros.org/wiki/xacro">
-    <xacro:include filename="$(find go2_description)/xacro/transmission.xacro"/>
+    <!-- <xacro:include filename="$(find go2_description)/transmission.xacro"/> -->
     <xacro:macro name="leg" params="name mirror mirror_dae front_hind front_hind_dae">
         <joint name="${name}_hip_joint" type="revolute">
@@ -17,5 +17,5 @@
             </xacro:if>
             <parent link="trunk"/>
-            <child link="${name}_hip"/>
+            <child link="${name}_hip_link"/>
             <axis xyz="1 0 0"/>
             <dynamics damping="${damping}" friction="${friction}"/>
@@ -27,5 +27,5 @@
             </xacro:if>
         </joint>
-        <link name="${name}_hip">
+        <link name="${name}_hip_link">
             <visual>
                 <xacro:if value="${(mirror_dae == True) and (front_hind_dae == True)}">
@@ -42,5 +42,5 @@
                 </xacro:if>
                 <geometry>
-                    <mesh filename="package://hip.dae" scale="1 1 1"/>
+                    <mesh filename="file://$(find go2_description)/meshes/hip.dae" scale="1 1 1"/>
                 </geometry>
                 <!-- <material name="orange"/> -->
@@ -61,21 +61,21 @@
             </inertial>
         </link>
-        <joint name="${name}_thigh_joint" type="revolute">
+        <joint name="${name}_upper_leg_joint" type="revolute">
             <origin rpy="0 0 0" xyz="0 ${thigh_offset*mirror} 0"/>
-            <parent link="${name}_hip"/>
-            <child link="${name}_thigh"/>
+            <parent link="${name}_hip_link"/>
+            <child link="${name}_upper_leg_link"/>
             <axis xyz="0 1 0"/>
             <dynamics damping="${damping}" friction="${friction}"/>
             <limit effort="${thigh_torque_max}" velocity="${thigh_velocity_max}" lower="${thigh_position_min}" upper="${thigh_position_max}"/>
         </joint>
-        <link name="${name}_thigh">
+        <link name="${name}_upper_leg_link">
             <visual>
                 <origin rpy="0 0 0" xyz="0 0 0"/>
                 <geometry>
                     <xacro:if value="${mirror_dae == True}">
-                        <mesh filename="package://thigh.dae" scale="1 1 1"/>
+                        <mesh filename="file://$(find go2_description)/meshes/thigh.dae" scale="1 1 1"/>
                     </xacro:if>
                     <xacro:if value="${mirror_dae == False}">
-                        <mesh filename="package://thigh_mirror.dae" scale="1 1 1"/>
+                        <mesh filename="file://$(find go2_description)/meshes/thigh_mirror.dae" scale="1 1 1"/>
                     </xacro:if>
                 </geometry>
@@ -97,17 +97,17 @@
             </inertial>
         </link>
-        <joint name="${name}_calf_joint" type="revolute">
+        <joint name="${name}_lower_leg_joint" type="revolute">
             <origin rpy="0 0 0" xyz="0 0 ${-thigh_length}"/>
-            <parent link="${name}_thigh"/>
-            <child link="${name}_calf"/>
+            <parent link="${name}_upper_leg_link"/>
+            <child link="${name}_lower_leg_link"/>
             <axis xyz="0 1 0"/>
             <dynamics damping="${damping}" friction="${friction}"/>
             <limit effort="${calf_torque_max}" velocity="${calf_velocity_max}" lower="${calf_position_min}" upper="${calf_position_max}"/>
         </joint>
-        <link name="${name}_calf">
+        <link name="${name}_lower_leg_link">
             <visual>
                 <origin rpy="0 0 0" xyz="0 0 0"/>
                 <geometry>
-                    <mesh filename="package://calf.dae" scale="1 1 1"/>
+                    <mesh filename="file://$(find go2_description)/meshes/calf.dae" scale="1 1 1"/>
                 </geometry>
                 <!-- <material name="orange"/> -->
@@ -128,10 +128,10 @@
             </inertial>
         </link>
-        <joint name="${name}_foot_fixed" type="fixed">
+        <joint name="${name}_foot_joint" type="fixed">0
             <origin rpy="0 0 0" xyz="0 0 ${-(calf_length)}"/>
-            <parent link="${name}_calf"/>
-            <child link="${name}_foot"/>
+            <parent link="${name}_lower_leg_link"/>
+            <child link="${name}_foot_link"/>
         </joint>
-        <link name="${name}_foot">
+        <link name="${name}_foot_link">
             <visual>
                 <origin rpy="0 0 0" xyz="0 0 0"/>
@@ -155,5 +155,25 @@
             </inertial>
         </link>
-        <xacro:leg_transmission name="${name}"/>
+        <ros2_control name="${name}" type="system">
+            <hardware>
+                <plugin>gz_ros2_control/GazeboSimSystem</plugin>
+            </hardware>
+            <joint name="${name}_hip_joint">
+                <command_interface name="position"/>
+                <state_interface name="position"/>
+                <state_interface name="velocity"/>
+            </joint>
+            <joint name="${name}_upper_leg_joint">
+                <command_interface name="position"/>
+                <state_interface name="position"/>
+                <state_interface name="velocity"/>
+            </joint>
+            <joint name="${name}_lower_leg_joint">
+                <command_interface name="position"/>
+                <state_interface name="position"/>
+                <state_interface name="velocity"/>
+            </joint>
+        </ros2_control>
+        <!-- <xacro:leg_transmission name="${name}"/> -->
     </xacro:macro>
 </robot>
