Commit message: Fix go2 naming issues and starting pose

File: go2_description/urdf/leg.xacro (robot description, xacro)
@@ -161,15 +161,21 @@
             <joint name="${name}_hip_joint">
                 <command_interface name="position"/>
-                <state_interface name="position"/>
+                <state_interface name="position">
+                  <param name="initial_value">0.0</param>
+                </state_interface>
                 <state_interface name="velocity"/>
             </joint>
             <joint name="${name}_upper_leg_joint">
                 <command_interface name="position"/>
-                <state_interface name="position"/>
+                <state_interface name="position">
+                  <param name="initial_value">0.5</param>
+                </state_interface>
                 <state_interface name="velocity"/>
             </joint>
             <joint name="${name}_lower_leg_joint">
                 <command_interface name="position"/>
-                <state_interface name="position"/>
+                <state_interface name="position">
+                  <param name="initial_value">-0.5</param>
+                </state_interface>
                 <state_interface name="velocity"/>
             </joint>

File: go2_description/urdf/unitree_go2_gazebo.xacro (robot description, xacro)
@@ -1,5 +1,5 @@
 <?xml version="1.0"?>
 <robot xmlns:xacro="http://ros.org/wiki/xacro">
-<xacro:macro name="unitree_go2_gazebo" params="robot_controllers">
+<xacro:macro name="unitree_go2_gazebo" params="robot_controllers robot_ns">
   <!-- Gazebo Sim plugins -->
   <gazebo>
@@ -28,172 +28,175 @@
       <parameters>${robot_controllers}</parameters>
       <robot_param_node>robot_state_publisher</robot_param_node>
+      <ros>
+        <namespace>${robot_ns}</namespace>
+      </ros>
     </plugin>
   </gazebo>
-        <!-- Odometry plugin -->
-        <gazebo>
-            <plugin filename="gz-sim-odometry-publisher-system"
-                name="gz::sim::systems::OdometryPublisher">
-                <odom_frame>odom</odom_frame>
-                <robot_base_frame>base_link</robot_base_frame>
-                <odom_topic>/odom</odom_topic>
-                <odom_publish_frequency>50</odom_publish_frequency>
+    <!-- Odometry plugin -->
+    <gazebo>
+        <plugin filename="gz-sim-odometry-publisher-system"
+            name="gz::sim::systems::OdometryPublisher">
+            <odom_frame>odom</odom_frame>
+            <robot_base_frame>base_link</robot_base_frame>
+            <odom_topic>${robot_ns}/odom</odom_topic>
+            <odom_publish_frequency>50</odom_publish_frequency>
+        </plugin>
+    </gazebo>
+    <!-- IMU plugin -->
+    <gazebo reference="imu_link">
+        <sensor name="imu_sensor" type="imu">
+            <always_on>true</always_on>
+            <update_rate>100</update_rate>
+            <visualize>true</visualize>
+            <topic>${robot_ns}/imu/data</topic>
+            <gz_frame_id>imu_link</gz_frame_id>
+            <imu>
+                <angular_velocity>
+                    <x>
+                        <noise type="gaussian">
+                            <mean>0.0</mean>
+                            <stddev>2e-4</stddev>
+                        </noise>
+                    </x>
+                    <y>
+                        <noise type="gaussian">
+                            <mean>0.0</mean>
+                            <stddev>2e-4</stddev>
+                        </noise>
+                    </y>
+                    <z>
+                        <noise type="gaussian">
+                            <mean>0.0</mean>
+                            <stddev>2e-4</stddev>
+                        </noise>
+                    </z>
+                </angular_velocity>
+                <linear_acceleration>
+                    <x>
+                        <noise type="gaussian">
+                            <mean>0.0</mean>
+                            <stddev>1.7e-2</stddev>
+                        </noise>
+                    </x>
+                    <y>
+                        <noise type="gaussian">
+                            <mean>0.0</mean>
+                            <stddev>1.7e-2</stddev>
+                        </noise>
+                    </y>
+                    <z>
+                        <noise type="gaussian">
+                            <mean>0.0</mean>
+                            <stddev>1.7e-2</stddev>
+                        </noise>
+                    </z>
+                </linear_acceleration>
+            </imu>
+            <plugin filename="gz-sim-imu-system" name="gz::sim::systems::Imu">
+                <initial_orientation_as_reference>false</initial_orientation_as_reference>
             </plugin>
-        </gazebo>
-        <!-- IMU plugin -->
-        <gazebo reference="imu_link">
-            <sensor name="imu_sensor" type="imu">
-                <always_on>true</always_on>
-                <update_rate>100</update_rate>
-                <visualize>true</visualize>
-                <topic>imu/data</topic>
-                <gz_frame_id>imu_link</gz_frame_id>
-                <imu>
-                    <angular_velocity>
-                        <x>
-                            <noise type="gaussian">
-                                <mean>0.0</mean>
-                                <stddev>2e-4</stddev>
-                            </noise>
-                        </x>
-                        <y>
-                            <noise type="gaussian">
-                                <mean>0.0</mean>
-                                <stddev>2e-4</stddev>
-                            </noise>
-                        </y>
-                        <z>
-                            <noise type="gaussian">
-                                <mean>0.0</mean>
-                                <stddev>2e-4</stddev>
-                            </noise>
-                        </z>
-                    </angular_velocity>
-                    <linear_acceleration>
-                        <x>
-                            <noise type="gaussian">
-                                <mean>0.0</mean>
-                                <stddev>1.7e-2</stddev>
-                            </noise>
-                        </x>
-                        <y>
-                            <noise type="gaussian">
-                                <mean>0.0</mean>
-                                <stddev>1.7e-2</stddev>
-                            </noise>
-                        </y>
-                        <z>
-                            <noise type="gaussian">
-                                <mean>0.0</mean>
-                                <stddev>1.7e-2</stddev>
-                            </noise>
-                        </z>
-                    </linear_acceleration>
-                </imu>
-                <plugin filename="gz-sim-imu-system" name="gz::sim::systems::Imu">
-                    <initial_orientation_as_reference>false</initial_orientation_as_reference>
-                </plugin>
-            </sensor>
-        </gazebo>
-        <!-- Camera Plugin-->
-        <gazebo reference="camera_link">
-            <sensor name="rgb_camera" type="camera">
-                <pose>0 0.0 0 0 0 0</pose>
-                <camera>
-                    <horizontal_fov>1.367</horizontal_fov>
-                    <image>
-                        <width>640</width>
-                        <height>480</height>
-                    </image>
-                    <clip>
-                        <near>0.05</near>
-                        <far>200</far>
-                    </clip>
-                </camera>
-                <gz_frame_id>camera_link</gz_frame_id>
-                <always_on>1</always_on>
-                <update_rate>10</update_rate>
-                <visualize>1</visualize>
-                <topic>rgb_image</topic>
-            </sensor>
-        </gazebo>
-        <!-- Main body -->
-        <gazebo reference="trunk">
-            <mu1>0.2</mu1>
-            <mu2>0.2</mu2>
-            <kp>10000.0</kp>
-            <kd>1.0</kd>
-        </gazebo>
-        <!-- FL leg -->
-        <gazebo reference="lf_hip_link">
-            <mu1>0.2</mu1>
-            <mu2>0.2</mu2>
-        </gazebo>
-        <gazebo reference="lf_upper_leg_link">
-            <mu1>0.2</mu1>
-            <mu2>0.2</mu2>
-            <self_collide>1</self_collide>
-            <kp>10000.0</kp>
-            <kd>1.0</kd>
-        </gazebo>
-        <gazebo reference="lf_lower_leg_link">
-            <mu1>0.2</mu1>
-            <mu2>0.2</mu2>
-            <self_collide>1</self_collide>
-        </gazebo>
-        <gazebo reference="lf_foot_link">
-            <mu1>0.6</mu1>
-            <mu2>0.6</mu2>
-            <self_collide>1</self_collide>
-            <kp>10000.0</kp>
-            <kd>1.0</kd>
-        </gazebo>
-        <!-- FR leg -->
-        <gazebo reference="rf_hip_link">
-            <mu1>0.2</mu1>
-            <mu2>0.2</mu2>
-        </gazebo>
-        <gazebo reference="rf_upper_leg_link">
-            <mu1>0.2</mu1>
-            <mu2>0.2</mu2>
-            <self_collide>1</self_collide>
-            <kp>10000.0</kp>
-            <kd>1.0</kd>
-        </gazebo>
-        <gazebo reference="rf_lower_leg_link">
-            <mu1>0.2</mu1>
-            <mu2>0.2</mu2>
-            <self_collide>1</self_collide>
-        </gazebo>
-        <gazebo reference="rf_foot_link">
-            <mu1>0.6</mu1>
-            <mu2>0.6</mu2>
-            <self_collide>1</self_collide>
-            <kp>10000.0</kp>
-            <kd>1.0</kd>
-        </gazebo>
-        <!-- RL leg -->
-        <gazebo reference="lh_hip_link">
-            <mu1>0.2</mu1>
-            <mu2>0.2</mu2>
-        </gazebo>
-        <gazebo reference="lh_upper_leg_link">
-            <mu1>0.2</mu1>
-            <mu2>0.2</mu2>
-            <self_collide>1</self_collide>
-            <kp>10000.0</kp>
-            <kd>1.0</kd>
-        </gazebo>
-        <gazebo reference="lh_lower_leg_link">
-            <mu1>0.2</mu1>
-            <mu2>0.2</mu2>
-            <self_collide>1</self_collide>
-        </gazebo>
-        <gazebo reference="lh_foot_link">
-            <mu1>0.6</mu1>
-            <mu2>0.6</mu2>
-            <self_collide>1</self_collide>
-            <kp>10000.0</kp>
-            <kd>1.0</kd>
-        </gazebo>
+        </sensor>
+    </gazebo>
+    <!-- Camera Plugin-->
+    <gazebo reference="camera_link">
+        <sensor name="rgb_camera" type="camera">
+            <pose>0 0.0 0 0 0 0</pose>
+            <camera>
+                <horizontal_fov>1.367</horizontal_fov>
+                <image>
+                    <width>640</width>
+                    <height>480</height>
+                </image>
+                <clip>
+                    <near>0.05</near>
+                    <far>200</far>
+                </clip>
+            </camera>
+            <gz_frame_id>camera_link</gz_frame_id>
+            <always_on>1</always_on>
+            <update_rate>10</update_rate>
+            <visualize>1</visualize>
+            <topic>${robot_ns}/rgb_image</topic>
+        </sensor>
+    </gazebo>
+    <!-- Main body -->
+    <gazebo reference="trunk">
+        <mu1>0.2</mu1>
+        <mu2>0.2</mu2>
+        <kp>10000.0</kp>
+        <kd>1.0</kd>
+    </gazebo>
+    <!-- FL leg -->
+    <gazebo reference="lf_hip_link">
+        <mu1>0.2</mu1>
+        <mu2>0.2</mu2>
+    </gazebo>
+    <gazebo reference="lf_upper_leg_link">
+        <mu1>0.2</mu1>
+        <mu2>0.2</mu2>
+        <self_collide>1</self_collide>
+        <kp>10000.0</kp>
+        <kd>1.0</kd>
+    </gazebo>
+    <gazebo reference="lf_lower_leg_link">
+        <mu1>0.2</mu1>
+        <mu2>0.2</mu2>
+        <self_collide>1</self_collide>
+    </gazebo>
+    <gazebo reference="lf_foot_link">
+        <mu1>0.6</mu1>
+        <mu2>0.6</mu2>
+        <self_collide>1</self_collide>
+        <kp>10000.0</kp>
+        <kd>1.0</kd>
+    </gazebo>
+    <!-- FR leg -->
+    <gazebo reference="rf_hip_link">
+        <mu1>0.2</mu1>
+        <mu2>0.2</mu2>
+    </gazebo>
+    <gazebo reference="rf_upper_leg_link">
+        <mu1>0.2</mu1>
+        <mu2>0.2</mu2>
+        <self_collide>1</self_collide>
+        <kp>10000.0</kp>
+        <kd>1.0</kd>
+    </gazebo>
+    <gazebo reference="rf_lower_leg_link">
+        <mu1>0.2</mu1>
+        <mu2>0.2</mu2>
+        <self_collide>1</self_collide>
+    </gazebo>
+    <gazebo reference="rf_foot_link">
+        <mu1>0.6</mu1>
+        <mu2>0.6</mu2>
+        <self_collide>1</self_collide>
+        <kp>10000.0</kp>
+        <kd>1.0</kd>
+    </gazebo>
+    <!-- RL leg -->
+    <gazebo reference="lh_hip_link">
+        <mu1>0.2</mu1>
+        <mu2>0.2</mu2>
+    </gazebo>
+    <gazebo reference="lh_upper_leg_link">
+        <mu1>0.2</mu1>
+        <mu2>0.2</mu2>
+        <self_collide>1</self_collide>
+        <kp>10000.0</kp>
+        <kd>1.0</kd>
+    </gazebo>
+    <gazebo reference="lh_lower_leg_link">
+        <mu1>0.2</mu1>
+        <mu2>0.2</mu2>
+        <self_collide>1</self_collide>
+    </gazebo>
+    <gazebo reference="lh_foot_link">
+        <mu1>0.6</mu1>
+        <mu2>0.6</mu2>
+        <self_collide>1</self_collide>
+        <kp>10000.0</kp>
+        <kd>1.0</kd>
+    </gazebo>
   <!-- RR leg -->
   <gazebo reference="rh_hip_link">

File: go2_description/urdf/unitree_go2_robot.xacro (robot description, xacro)
@@ -4,4 +4,5 @@
     <xacro:arg name="DEBUG" default="false"/>
     <xacro:arg name="robot_controllers" default="$(find go2_description)/config/ros_control/ros_control.yaml"/>
+    <xacro:arg name="robot_ns" default=""/>
     <xacro:include filename="$(find go2_description)/urdf/const.xacro" />
     <xacro:include filename="$(find go2_description)/urdf/materials.xacro" />
@@ -14,5 +15,5 @@
     <xacro:include filename="$(find go2_description)/urdf/realsense_d455.xacro"/>
     <!-- <xacro:stairs stairs="15" xpos="0" ypos="0" zpos="0" /> -->
-    <xacro:unitree_go2_gazebo robot_controllers="$(arg robot_controllers)"/>
+    <xacro:unitree_go2_gazebo robot_controllers="$(arg robot_controllers)" robot_ns="$(arg robot_ns)"/>
     <!-- Rotor related joint and link is only for demonstrate location. -->
     <!-- Actually, the rotor will rotate and the joint is not fixed. Reduction ratio should be
