Commit message: adds multimodal robot and improves go2 spawning

File: ros2_gz_sandbox/urdf/multimodal.urdf.xacro (robot description, xacro)
@@ -24,6 +24,6 @@
     </collision>
     <inertial>
-      <mass value="0.1"/>
-      <inertia ixx="0.2" ixy="0.0" ixz="0.0" iyy="0.2" iyz="0.0" izz="0.2"/>
+      <mass value="1.0"/>
+      <inertia ixx="0.002" ixy="0.0" ixz="0.0" iyy="0.002" iyz="0.0" izz="0.002"/>
     </inertial>
   </link>
@@ -47,5 +47,5 @@
       <inertial>
         <mass value="0.1"/>
-        <inertia ixx="0.01" ixy="0.0" ixz="0.0" iyy="0.01" iyz="0.0" izz="0.01"/>
+        <inertia ixx="0.001" ixy="0.0" ixz="0.0" iyy="0.001" iyz="0.0" izz="0.001"/>
       </inertial>
     </link>
@@ -123,6 +123,6 @@
     </collision>
     <inertial>
-      <mass value="0.1"/>
-      <inertia ixx="0.01" ixy="0.0" ixz="0.0" iyy="0.01" iyz="0.0" izz="0.01"/>
+      <mass value="0.001"/>
+      <inertia ixx="0.0001" ixy="0.0" ixz="0.0" iyy="0.0001" iyz="0.0" izz="0.0001"/>
     </inertial>
   </link>
@@ -162,5 +162,5 @@
       <update_rate>30</update_rate>
       <visualize>true</visualize>
-      <topic>camera/image_raw</topic>
+      <topic>${robot_ns}/camera/image_raw</topic>
       <gz_frame_id>camera_link</gz_frame_id>
     </sensor>
@@ -169,5 +169,5 @@
     <sensor name="lidar_link" type="gpu_lidar">
     <pose>0 0 0 0 0 0</pose>
-      <topic>pointcloud</topic>
+      <topic>${robot_ns}/pointcloud</topic>
       <update_rate>10</update_rate>
       <ray>
@@ -329,5 +329,5 @@
         <odom_topic>${robot_ns}/true_pose</odom_topic>
         <odom_frame>odom</odom_frame>
-        <dimensions>2</dimensions>
+        <dimensions>3</dimensions>
         <robot_base_frame>base_link</robot_base_frame>
         <tf_topic>${robot_ns}/tf</tf_topic>
